Commit message: added headless and updated readme

File: output/label29.urdf (robot description, URDF)
Before this commit: robot my_urdf, 9 links, 8 joints
Joints:
- joint knob4_to_drawer0: limit lower=-1.57 upper=0 effort=5 velocity=2.283 -> lower=0 upper=1.57 effort=5 velocity=2.283
- joint knob5_to_drawer1: limit lower=-1.57 upper=0 effort=5 velocity=2.283 -> lower=0 upper=1.57 effort=5 velocity=2.283
- joint knob6_to_doorR2: limit lower=-1.57 upper=0 effort=5 velocity=2.283 -> lower=0 upper=1.57 effort=5 velocity=2.283
- joint knob7_to_doorL3: limit lower=-1.57 upper=0 effort=5 velocity=2.283 -> lower=0 upper=1.57 effort=5 velocity=2.283

File: output/label31.urdf (robot description, URDF)
Before this commit: robot my_urdf, 7 links, 6 joints
Joints:
- joint knob3_to_drawer0: limit lower=-1.57 upper=0 effort=5 velocity=2.283 -> lower=0 upper=1.57 effort=5 velocity=2.283
- joint knob4_to_doorR1: limit lower=-1.57 upper=0 effort=5 velocity=2.283 -> lower=0 upper=1.57 effort=5 velocity=2.283
- joint knob5_to_doorL2: limit lower=-1.57 upper=0 effort=5 velocity=2.283 -> lower=0 upper=1.57 effort=5 velocity=2.283

File: output/label53.urdf (robot description, URDF)
Before this commit: robot my_urdf, 11 links, 10 joints
Joints:
- joint handle5_to_drawer0: limit lower=-1.57 upper=0 effort=5 velocity=2.283 -> lower=0 upper=1.57 effort=5 velocity=2.283
- joint handle6_to_drawer1: limit lower=-1.57 upper=0 effort=5 velocity=2.283 -> lower=0 upper=1.57 effort=5 velocity=2.283
- joint handle7_to_drawer2: limit lower=-1.57 upper=0 effort=5 velocity=2.283 -> lower=0 upper=1.57 effort=5 velocity=2.283
- joint handle8_to_drawer3: limit lower=-1.57 upper=0 effort=5 velocity=2.283 -> lower=0 upper=1.57 effort=5 velocity=2.283
- joint handle9_to_doorL4: limit lower=-1.57 upper=0 effort=5 velocity=2.283 -> lower=0 upper=1.57 effort=5 velocity=2.283

File: output/label62.urdf (robot description, URDF)
Before this commit: robot my_urdf, 7 links, 6 joints
Joints:
- joint knob3_to_drawer0: limit lower=0 upper=0.4 effort=5 velocity=2.283 -> lower=0 upper=1.57 effort=5 velocity=2.283
- joint knob4_to_drawer1: limit lower=0 upper=0.4 effort=5 velocity=2.283 -> lower=0 upper=1.57 effort=5 velocity=2.283
- joint knob5_to_drawer2: limit lower=0 upper=0.4 effort=5 velocity=2.283 -> lower=0 upper=1.57 effort=5 velocity=2.283
